File: Kicad/maquina_compostaje/A3144.kicad_sch (KiCad schematic)
At the start: 9 parts, among them U8 LM393, U9 A3144

Commit message: inicio del ruteo
Connections:
- net +5V is gone; now on net 5v: RV1.1
Changed lines of the file:
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@@
     (effects (font (size 2.4892 2.4892)) (justify left bottom))
+  )
+  (hierarchical_label "5v" (shape input) (at 152.4 107.95 90)
+    (effects (font (size 1.27 1.27)) (justify left))
   )
   (hierarchical_label "5v" (shape input) (at 97.79 73.66 90)
@@
     (pin "2")
   )
-  (symbol (lib_id "power:+5V") (at 152.4 107.95 0) (unit 1)
-    (in_bom yes) (on_board yes)
-    (property "Reference" "#PWR0102" (id 0) (at 152.4 111.76 0)
-      (effects (font (size 1.27 1.27)) hide)
-    )
-    (property "Value" "+5V" (id 1) (at 152.781 103.5558 0))
-    (property "Footprint" "" (id 2) (at 152.4 107.95 0)
-      (effects (font (size 1.27 1.27)) hide)
-    )
-    (property "Datasheet" "" (id 3) (at 152.4 107.95 0)
-      (effects (font (size 1.27 1.27)) hide)
-    )
-    (pin "1")
-  )
   (symbol (lib_id "power:GND") (at 152.4 121.92 0) (unit 1)
