File: Kicad/maquina_compostaje/Motor A.kicad_sch (KiCad schematic)
At the start: 12 parts, among them J3 Conn_01x04, U4 L298N

Commit message: inicio del ruteo
Parts:
- added R33, R34: 4.7K, Resistor_SMD:R_1206_3216Metric_Pad1.30x1.75mm_HandSolder, symbol Device:R
- D1, D2, D3, D4, D5, D6, D7, D8: footprint M7:DIOM505270X240 -> Diode_SMD:D_SOD-128
Connections:
- net EN_1A: now also R33.2
- net EN_2A: now also R34.1
- net GND: now also R33.1, R34.2
Changed lines of the file:
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@@
   (junction (at 154.94 68.58) (diameter 0) (color 0 0 0 0)
   )
+  (junction (at 83.82 93.98) (diameter 0) (color 0 0 0 0)
+  )
+  (junction (at 83.82 81.28) (diameter 0) (color 0 0 0 0)
+  )
   (junction (at 170.18 93.98) (diameter 0) (color 0 0 0 0)
   )
@@
     (stroke (width 0) (type default) (color 0 0 0 0))
   )
+  (wire (pts (xy 83.82 93.98) (xy 91.44 93.98))
+    (stroke (width 0) (type default) (color 0 0 0 0))
+  )
   (wire (pts (xy 102.87 85.09) (xy 90.17 85.09))
     (stroke (width 0) (type default) (color 0 0 0 0))
@@
     (stroke (width 0) (type default) (color 0 0 0 0))
   )
-  (wire (pts (xy 90.17 81.28) (xy 71.12 81.28))
+  (wire (pts (xy 90.17 81.28) (xy 83.82 81.28))
     (stroke (width 0) (type default) (color 0 0 0 0))
   )
@@
     (stroke (width 0) (type default) (color 0 0 0 0))
   )
-  (wire (pts (xy 91.44 93.98) (xy 71.12 93.98))
+  (wire (pts (xy 71.12 93.98) (xy 83.82 93.98))
+    (stroke (width 0) (type default) (color 0 0 0 0))
+  )
+  (wire (pts (xy 83.82 96.52) (xy 83.82 93.98))
     (stroke (width 0) (type default) (color 0 0 0 0))
   )
@@
     (stroke (width 0) (type default) (color 0 0 0 0))
   )
+  (wire (pts (xy 83.82 81.28) (xy 71.12 81.28))
+    (stroke (width 0) (type default) (color 0 0 0 0))
+  )
   (wire (pts (xy 154.94 107.95) (xy 154.94 115.57))
     (stroke (width 0) (type default) (color 0 0 0 0))
@@
     (stroke (width 0) (type default) (color 0 0 0 0))
   )
+  (wire (pts (xy 83.82 71.12) (xy 83.82 66.04))
+    (stroke (width 0) (type default) (color 0 0 0 0))
+  )
   (wire (pts (xy 144.78 59.69) (xy 144.78 68.58))
     (stroke (width 0) (type default) (color 0 0 0 0))
@@
     (stroke (width 0) (type default) (color 0 0 0 0))
   )
+  (wire (pts (xy 91.44 106.68) (xy 91.44 104.14))
+    (stroke (width 0) (type default) (color 0 0 0 0))
+  )
   (wire (pts (xy 170.18 93.98) (xy 205.74 93.98))
     (stroke (width 0) (type default) (color 0 0 0 0))
@@
     (stroke (width 0) (type default) (color 0 0 0 0))
   )
+  (wire (pts (xy 91.44 66.04) (xy 91.44 68.58))
+    (stroke (width 0) (type default) (color 0 0 0 0))
+  )
   (wire (pts (xy 162.56 68.58) (xy 170.18 68.58))
     (stroke (width 0) (type default) (color 0 0 0 0))
@@
     (stroke (width 0) (type default) (color 0 0 0 0))
   )
+  (wire (pts (xy 83.82 78.74) (xy 83.82 81.28))
+    (stroke (width 0) (type default) (color 0 0 0 0))
+  )
   (wire (pts (xy 170.18 107.95) (xy 170.18 115.57))
     (stroke (width 0) (type default) (color 0 0 0 0))
@@
     (stroke (width 0) (type default) (color 0 0 0 0))
   )
+  (wire (pts (xy 83.82 104.14) (xy 91.44 104.14))
+    (stroke (width 0) (type default) (color 0 0 0 0))
+  )
   (polyline (pts (xy 54.61 48.26) (xy 54.61 66.04))
     (stroke (width 0) (type default) (color 0 0 0 0))
@@
   )
   (wire (pts (xy 110.49 115.57) (xy 113.03 115.57))
+    (stroke (width 0) (type default) (color 0 0 0 0))
+  )
+  (wire (pts (xy 83.82 66.04) (xy 91.44 66.04))
     (stroke (width 0) (type default) (color 0 0 0 0))
   )
@@
       (effects (font (size 1.27 1.27)) (justify left))
     )
-    (property "Footprint" "M7:DIOM505270X240" (id 2) (at 158.115 72.39 0)
+    (property "Footprint" "Diode_SMD:D_SOD-128" (id 2) (at 158.115 72.39 0)
       (effects (font (size 1.27 1.27)) hide)
     )
@@
     )
     (property "Datasheet" "~" (id 3) (at 111.76 63.5 0)
+      (effects (font (size 1.27 1.27)) hide)
+    )
+    (pin "1")
+    (pin "2")
+  )
+  (symbol (lib_id "Device:R") (at 83.82 100.33 0) (unit 1)
+    (in_bom yes) (on_board yes) (fields_autoplaced)
+    (property "Reference" "R34" (id 0) (at 86.36 99.0599 0)
+      (effects (font (size 1.27 1.27)) (justify left))
+    )
+    (property "Value" "4.7K" (id 1) (at 86.36 101.5999 0)
+      (effects (font (size 1.27 1.27)) (justify left))
+    )
+    (property "Footprint" "Resistor_SMD:R_1206_3216Metric_Pad1.30x1.75mm_HandSolder" (id 2) (at 82.042 100.33 90)
+      (effects (font (size 1.27 1.27)) hide)
+    )
+    (property "Datasheet" "~" (id 3) (at 83.82 100.33 0)
       (effects (font (size 1.27 1.27)) hide)
     )
@@
     (pin "4")
   )
+  (symbol (lib_id "Device:R") (at 83.82 74.93 0) (unit 1)
+    (in_bom yes) (on_board yes) (fields_autoplaced)
+    (property "Reference" "R33" (id 0) (at 86.36 73.6599 0)
+      (effects (font (size 1.27 1.27)) (justify left))
+    )
+    (property "Value" "4.7K" (id 1) (at 86.36 76.1999 0)
+      (effects (font (size 1.27 1.27)) (justify left))
+    )
+    (property "Footprint" "Resistor_SMD:R_1206_3216Metric_Pad1.30x1.75mm_HandSolder" (id 2) (at 82.042 74.93 90)
+      (effects (font (size 1.27 1.27)) hide)
+    )
+    (property "Datasheet" "~" (id 3) (at 83.82 74.93 0)
+      (effects (font (size 1.27 1.27)) hide)
+    )
+    (pin "1")
+    (pin "2")
+  )
   (symbol (lib_id "power:GND") (at 191.77 80.01 0) (unit 1)
     (in_bom yes) (on_board yes) (fields_autoplaced)
@@
       (effects (font (size 1.27 1.27)) (justify left))
     )
-    (property "Footprint" "M7:DIOM505270X240" (id 2) (at 150.495 72.39 0)
+    (property "Footprint" "Diode_SMD:D_SOD-128" (id 2) (at 150.495 72.39 0)
       (effects (font (size 1.27 1.27)) hide)
     )
@@
     (pin "1")
     (pin "2")
+  )
+  (symbol (lib_id "power:GND") (at 91.44 106.68 0) (unit 1)
+    (in_bom yes) (on_board yes) (fields_autoplaced)
+    (property "Reference" "#PWR03" (id 0) (at 91.44 113.03 0)
+      (effects (font (size 1.27 1.27)) hide)
+    )
+    (property "Value" "GND" (id 1) (at 91.44 111.76 0))
+    (property "Footprint" "" (id 2) (at 91.44 106.68 0)
+      (effects (font (size 1.27 1.27)) hide)
+    )
+    (property "Datasheet" "" (id 3) (at 91.44 106.68 0)
+      (effects (font (size 1.27 1.27)) hide)
+    )
+    (pin "1")
   )
   (symbol (lib_id "Driver_Motor:L298N") (at 118.11 92.71 0) (unit 1)
@@
     (pin "9")
   )
+  (symbol (lib_id "power:GND") (at 91.44 68.58 0) (unit 1)
+    (in_bom yes) (on_board yes) (fields_autoplaced)
+    (property "Reference" "#PWR02" (id 0) (at 91.44 74.93 0)
+      (effects (font (size 1.27 1.27)) hide)
+    )
+    (property "Value" "GND" (id 1) (at 91.44 73.66 0))
+    (property "Footprint" "" (id 2) (at 91.44 68.58 0)
+      (effects (font (size 1.27 1.27)) hide)
+    )
+    (property "Datasheet" "" (id 3) (at 91.44 68.58 0)
+      (effects (font (size 1.27 1.27)) hide)
+    )
+    (pin "1")
+  )
   (symbol (lib_id "Diode:1N4007") (at 154.94 104.14 270) (unit 1)
     (in_bom yes) (on_board yes)
@@
       (effects (font (size 1.27 1.27)) (justify left))
     )
-    (property "Footprint" "M7:DIOM505270X240" (id 2) (at 150.495 104.14 0)
+    (property "Footprint" "Diode_SMD:D_SOD-128" (id 2) (at 150.495 104.14 0)
       (effects (font (size 1.27 1.27)) hide)
     )
@@
       (effects (font (size 1.27 1.27)) (justify left))
     )
-    (property "Footprint" "M7:DIOM505270X240" (id 2) (at 173.355 72.39 0)
+    (property "Footprint" "Diode_SMD:D_SOD-128" (id 2) (at 173.355 72.39 0)
       (effects (font (size 1.27 1.27)) hide)
     )
@@
       (effects (font (size 1.27 1.27)) (justify left))
     )
-    (property "Footprint" "M7:DIOM505270X240" (id 2) (at 173.355 104.14 0)
+    (property "Footprint" "Diode_SMD:D_SOD-128" (id 2) (at 173.355 104.14 0)
       (effects (font (size 1.27 1.27)) hide)
     )
@@
       (effects (font (size 1.27 1.27)) (justify left))
     )
-    (property "Footprint" "M7:DIOM505270X240" (id 2) (at 158.115 104.14 0)
+    (property "Footprint" "Diode_SMD:D_SOD-128" (id 2) (at 158.115 104.14 0)
       (effects (font (size 1.27 1.27)) hide)
     )
@@
       (effects (font (size 1.27 1.27)) (justify left))
     )
-    (property "Footprint" "M7:DIOM505270X240" (id 2) (at 165.735 104.14 0)
+    (property "Footprint" "Diode_SMD:D_SOD-128" (id 2) (at 165.735 104.14 0)
       (effects (font (size 1.27 1.27)) hide)
     )
@@
       (effects (font (size 1.27 1.27)) (justify left))
     )
-    (property "Footprint" "M7:DIOM505270X240" (id 2) (at 165.735 72.39 0)
-      (effects (font (size 1.27 1.27)) hide)
-    )
+    (property "Footprint" "Diode_SMD:D_SOD-128" (id 2) (at 165.735 72.39 0)
+      (effects (font (size 1.27 1.27)) hide)
+    )
