File: Kicad/maquina_compostaje/Motor B.kicad_sch (KiCad schematic)
At the start: 12 parts, among them J4 Conn_01x04, U5 L298N

Commit message: inicio del ruteo
Parts:
- added R35, R36: 4.7K, Resistor_SMD:R_1206_3216Metric_Pad1.30x1.75mm_HandSolder, symbol Device:R
- D10, D11, D12, D13, D14, D15, D16, D9: footprint M7:DIOM505270X240 -> Diode_SMD:D_SOD-128
Connections:
- net EN_1B: now also R35.2
- net EN_2B: now also R36.1
- net GND: now also R35.1, R36.2
- net 1B renamed B1
- net 2B renamed B2
- net 3B renamed B3
- net 4B renamed B4
Changed lines of the file:
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@@
   (junction (at 115.57 64.77) (diameter 0) (color 0 0 0 0)
   )
+  (junction (at 90.17 87.63) (diameter 0) (color 0 0 0 0)
+  )
+  (junction (at 90.17 100.33) (diameter 0) (color 0 0 0 0)
+  )
   (junction (at 171.45 121.92) (diameter 0) (color 0 0 0 0)
   )
@@
     (stroke (width 0) (type default) (color 0 0 0 0))
   )
+  (wire (pts (xy 100.33 111.76) (xy 90.17 111.76))
+    (stroke (width 0) (type default) (color 0 0 0 0))
+  )
   (wire (pts (xy 158.75 74.93) (xy 166.37 74.93))
     (stroke (width 0) (type default) (color 0 0 0 0))
@@
     (stroke (width 0) (type default) (color 0 0 0 0))
   )
+  (wire (pts (xy 90.17 100.33) (xy 74.93 100.33))
+    (stroke (width 0) (type default) (color 0 0 0 0))
+  )
   (wire (pts (xy 97.79 97.79) (xy 74.93 97.79))
     (stroke (width 0) (type default) (color 0 0 0 0))
@@
     (stroke (width 0) (type default) (color 0 0 0 0))
   )
+  (wire (pts (xy 90.17 100.33) (xy 90.17 104.14))
+    (stroke (width 0) (type default) (color 0 0 0 0))
+  )
   (wire (pts (xy 114.3 116.84) (xy 114.3 121.92))
     (stroke (width 0) (type default) (color 0 0 0 0))
@@
     (stroke (width 0) (type default) (color 0 0 0 0))
   )
+  (wire (pts (xy 90.17 87.63) (xy 74.93 87.63))
+    (stroke (width 0) (type default) (color 0 0 0 0))
+  )
   (wire (pts (xy 181.61 102.87) (xy 209.55 102.87))
     (stroke (width 0) (type default) (color 0 0 0 0))
@@
     (stroke (width 0) (type default) (color 0 0 0 0))
   )
-  (wire (pts (xy 93.98 87.63) (xy 74.93 87.63))
+  (wire (pts (xy 93.98 87.63) (xy 90.17 87.63))
     (stroke (width 0) (type default) (color 0 0 0 0))
   )
@@
     (stroke (width 0) (type default) (color 0 0 0 0))
   )
+  (wire (pts (xy 90.17 82.55) (xy 90.17 87.63))
+    (stroke (width 0) (type default) (color 0 0 0 0))
+  )
   (wire (pts (xy 173.99 114.3) (xy 173.99 121.92))
     (stroke (width 0) (type default) (color 0 0 0 0))
@@
     (stroke (width 0) (type default) (color 0 0 0 0))
   )
+  (wire (pts (xy 90.17 67.31) (xy 100.33 67.31))
+    (stroke (width 0) (type default) (color 0 0 0 0))
+  )
   (polyline (pts (xy 233.68 54.61) (xy 58.42 54.61))
     (stroke (width 0) (type default) (color 0 0 0 0))
@@
     (stroke (width 0) (type default) (color 0 0 0 0))
   )
-  (wire (pts (xy 95.25 100.33) (xy 74.93 100.33))
+  (wire (pts (xy 95.25 100.33) (xy 90.17 100.33))
     (stroke (width 0) (type default) (color 0 0 0 0))
   )
@@
     (stroke (width 0) (type default) (color 0 0 0 0))
   )
+  (wire (pts (xy 100.33 67.31) (xy 100.33 69.85))
+    (stroke (width 0) (type default) (color 0 0 0 0))
+  )
+  (wire (pts (xy 100.33 115.57) (xy 100.33 111.76))
+    (stroke (width 0) (type default) (color 0 0 0 0))
+  )
   (wire (pts (xy 181.61 102.87) (xy 181.61 106.68))
     (stroke (width 0) (type default) (color 0 0 0 0))
@@
     (stroke (width 0) (type default) (color 0 0 0 0))
   )
+  (wire (pts (xy 90.17 74.93) (xy 90.17 67.31))
+    (stroke (width 0) (type default) (color 0 0 0 0))
+  )
   (wire (pts (xy 181.61 114.3) (xy 181.61 121.92))
     (stroke (width 0) (type default) (color 0 0 0 0))
@@
     (effects (font (size 1.27 1.27)) (justify left bottom))
   )
-  (hierarchical_label "4B" (shape input) (at 74.93 97.79 180)
+  (hierarchical_label "B4" (shape input) (at 74.93 97.79 180)
     (effects (font (size 1.27 1.27)) (justify right))
   )
@@
     (effects (font (size 1.27 1.27)) (justify left))
   )
-  (hierarchical_label "1B" (shape input) (at 74.93 90.17 180)
+  (hierarchical_label "B1" (shape input) (at 74.93 90.17 180)
     (effects (font (size 1.27 1.27)) (justify right))
   )
-  (hierarchical_label "3B" (shape input) (at 74.93 95.25 180)
+  (hierarchical_label "B3" (shape input) (at 74.93 95.25 180)
     (effects (font (size 1.27 1.27)) (justify right))
   )
@@
     (effects (font (size 1.27 1.27)) (justify left))
   )
-  (hierarchical_label "2B" (shape input) (at 74.93 92.71 180)
+  (hierarchical_label "B2" (shape input) (at 74.93 92.71 180)
     (effects (font (size 1.27 1.27)) (justify right))
   )
@@
     (effects (font (size 1.27 1.27)) (justify right))
   )
+  (symbol (lib_id "Device:R") (at 90.17 107.95 0) (unit 1)
+    (in_bom yes) (on_board yes) (fields_autoplaced)
+    (property "Reference" "R36" (id 0) (at 92.71 106.6799 0)
+      (effects (font (size 1.27 1.27)) (justify left))
+    )
+    (property "Value" "4.7K" (id 1) (at 92.71 109.2199 0)
+      (effects (font (size 1.27 1.27)) (justify left))
+    )
+    (property "Footprint" "Resistor_SMD:R_1206_3216Metric_Pad1.30x1.75mm_HandSolder" (id 2) (at 88.392 107.95 90)
+      (effects (font (size 1.27 1.27)) hide)
+    )
+    (property "Datasheet" "~" (id 3) (at 90.17 107.95 0)
+      (effects (font (size 1.27 1.27)) hide)
+    )
+    (pin "1")
+    (pin "2")
+  )
   (symbol (lib_id "Diode:1N4007") (at 158.75 110.49 270) (unit 1)
     (in_bom yes) (on_board yes)
@@
       (effects (font (size 1.27 1.27)) (justify left))
     )
-    (property "Footprint" "M7:DIOM505270X240" (id 2) (at 154.305 110.49 0)
+    (property "Footprint" "Diode_SMD:D_SOD-128" (id 2) (at 154.305 110.49 0)
       (effects (font (size 1.27 1.27)) hide)
     )
@@
       (effects (font (size 1.27 1.27)) (justify left))
     )
-    (property "Footprint" "M7:DIOM505270X240" (id 2) (at 154.305 78.74 0)
+    (property "Footprint" "Diode_SMD:D_SOD-128" (id 2) (at 154.305 78.74 0)
       (effects (font (size 1.27 1.27)) hide)
     )
@@
       (effects (font (size 1.27 1.27)) (justify left))
     )
-    (property "Footprint" "M7:DIOM505270X240" (id 2) (at 177.165 78.74 0)
+    (property "Footprint" "Diode_SMD:D_SOD-128" (id 2) (at 177.165 78.74 0)
       (effects (font (size 1.27 1.27)) hide)
     )
@@
       (effects (font (size 1.27 1.27)) (justify left))
     )
-    (property "Footprint" "M7:DIOM505270X240" (id 2) (at 177.165 110.49 0)
+    (property "Footprint" "Diode_SMD:D_SOD-128" (id 2) (at 177.165 110.49 0)
       (effects (font (size 1.27 1.27)) hide)
     )
@@
       (effects (font (size 1.27 1.27)) (justify left))
     )
-    (property "Footprint" "M7:DIOM505270X240" (id 2) (at 161.925 78.74 0)
+    (property "Footprint" "Diode_SMD:D_SOD-128" (id 2) (at 161.925 78.74 0)
       (effects (font (size 1.27 1.27)) hide)
     )
@@
       (effects (font (size 1.27 1.27)) (justify left))
     )
-    (property "Footprint" "M7:DIOM505270X240" (id 2) (at 161.925 110.49 0)
+    (property "Footprint" "Diode_SMD:D_SOD-128" (id 2) (at 161.925 110.49 0)
       (effects (font (size 1.27 1.27)) hide)
     )
@@
     (pin "1")
   )
+  (symbol (lib_id "power:GND") (at 100.33 69.85 0) (unit 1)
+    (in_bom yes) (on_board yes) (fields_autoplaced)
+    (property "Reference" "#PWR04" (id 0) (at 100.33 76.2 0)
+      (effects (font (size 1.27 1.27)) hide)
+    )
+    (property "Value" "GND" (id 1) (at 100.33 74.93 0))
+    (property "Footprint" "" (id 2) (at 100.33 69.85 0)
+      (effects (font (size 1.27 1.27)) hide)
+    )
+    (property "Datasheet" "" (id 3) (at 100.33 69.85 0)
+      (effects (font (size 1.27 1.27)) hide)
+    )
+    (pin "1")
+  )
   (symbol (lib_id "power:GND") (at 195.58 86.36 0) (unit 1)
     (in_bom yes) (on_board yes) (fields_autoplaced)
@@
     (pin "1")
   )
+  (symbol (lib_id "power:GND") (at 100.33 115.57 0) (unit 1)
+    (in_bom yes) (on_board yes) (fields_autoplaced)
+    (property "Reference" "#PWR05" (id 0) (at 100.33 121.92 0)
+      (effects (font (size 1.27 1.27)) hide)
+    )
+    (property "Value" "GND" (id 1) (at 100.33 120.65 0))
+    (property "Footprint" "" (id 2) (at 100.33 115.57 0)
+      (effects (font (size 1.27 1.27)) hide)
+    )
+    (property "Datasheet" "" (id 3) (at 100.33 115.57 0)
+      (effects (font (size 1.27 1.27)) hide)
+    )
+    (pin "1")
+  )
   (symbol (lib_id "Diode:1N4007") (at 173.99 78.74 270) (unit 1)
     (in_bom yes) (on_board yes)
@@
       (effects (font (size 1.27 1.27)) (justify left))
     )
-    (property "Footprint" "M7:DIOM505270X240" (id 2) (at 169.545 78.74 0)
+    (property "Footprint" "Diode_SMD:D_SOD-128" (id 2) (at 169.545 78.74 0)
       (effects (font (size 1.27 1.27)) hide)
     )
@@
     (pin "2")
   )
+  (symbol (lib_id "Device:R") (at 90.17 78.74 0) (unit 1)
+    (in_bom yes) (on_board yes) (fields_autoplaced)
+    (property "Reference" "R35" (id 0) (at 92.71 77.4699 0)
+      (effects (font (size 1.27 1.27)) (justify left))
+    )
+    (property "Value" "4.7K" (id 1) (at 92.71 80.0099 0)
+      (effects (font (size 1.27 1.27)) (justify left))
+    )
+    (property "Footprint" "Resistor_SMD:R_1206_3216Metric_Pad1.30x1.75mm_HandSolder" (id 2) (at 88.392 78.74 90)
+      (effects (font (size 1.27 1.27)) hide)
+    )
+    (property "Datasheet" "~" (id 3) (at 90.17 78.74 0)
+      (effects (font (size 1.27 1.27)) hide)
+    )
+    (pin "1")
+    (pin "2")
+  )
   (symbol (lib_id "Diode:1N4007") (at 173.99 110.49 270) (unit 1)
     (in_bom yes) (on_board yes)
@@
       (effects (font (size 1.27 1.27)) (justify left))
     )
-    (property "Footprint" "M7:DIOM505270X240" (id 2) (at 169.545 110.49 0)
-      (effects (font (size 1.27 1.27)) hide)
-    )
+    (property "Footprint" "Diode_SMD:D_SOD-128" (id 2) (at 169.545 110.49 0)
+      (effects (font (size 1.27 1.27)) hide)
+    )
