File: Kicad/maquina_compostaje/Opto.kicad_sch (KiCad schematic)
At the start: 17 parts, among them Q1 BC328, Q2 BC328, Q3 BC328, Q4 BC328, U2 TLP281-4GB(F)

Commit message: inicio del ruteo
Parts:
- Q1, Q2, Q3, Q4: footprint Package_TO_SOT_THT:TO-92_Inline -> Package_TO_SOT_SMD:SOT-23
- U2: footprint (none) -> Package_SO:SO-16_5.3x10.2mm_P1.27mm
Changed lines of the file:
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@@
-    (stroke (width 0) (type default) (color 0 0 0 0))
-  )
-  (wire (pts (xy 157.48 29.21) (xy 182.88 29.21))
     (stroke (width 0) (type default) (color 0 0 0 0))
   )
@@
   )
   (hierarchical_label "A3" (shape output) (at 182.88 67.31 0)
-    (effects (font (size 1.27 1.27)) (justify left))
-  )
-  (hierarchical_label "Vo_12V" (shape output) (at 182.88 29.21 0)
     (effects (font (size 1.27 1.27)) (justify left))
   )
@@
       (effects (font (size 1.27 1.27)) (justify left))
     )
-    (property "Footprint" "Package_TO_SOT_THT:TO-92_Inline" (id 2) (at 160.02 53.975 0)
+    (property "Footprint" "Package_TO_SOT_SMD:SOT-23" (id 2) (at 160.02 53.975 0)
       (effects (font (size 1.27 1.27) italic) (justify left) hide)
     )
@@
     (property "Reference" "U2" (id 0) (at 69.85 45.2882 0))
     (property "Value" "TLP281-4GB(F)" (id 1) (at 69.85 47.5996 0))
-    (property "Footprint" "" (id 2) (at 68.58 69.85 0)
+    (property "Footprint" "Package_SO:SO-16_5.3x10.2mm_P1.27mm" (id 2) (at 68.58 69.85 0)
       (effects (font (size 1.27 1.27)) (justify left bottom) hide)
     )
@@
       (effects (font (size 1.27 1.27)) (justify left))
     )
-    (property "Footprint" "Package_TO_SOT_THT:TO-92_Inline" (id 2) (at 102.87 84.455 0)
+    (property "Footprint" "Package_TO_SOT_SMD:SOT-23" (id 2) (at 102.87 84.455 0)
       (effects (font (size 1.27 1.27) italic) (justify left) hide)
     )
@@
       (effects (font (size 1.27 1.27)) (justify left))
     )
-    (property "Footprint" "Package_TO_SOT_THT:TO-92_Inline" (id 2) (at 140.97 64.135 0)
+    (property "Footprint" "Package_TO_SOT_SMD:SOT-23" (id 2) (at 140.97 64.135 0)
       (effects (font (size 1.27 1.27) italic) (justify left) hide)
     )
@@
       (effects (font (size 1.27 1.27)) (justify left))
     )
-    (property "Footprint" "Package_TO_SOT_THT:TO-92_Inline" (id 2) (at 121.92 74.295 0)
+    (property "Footprint" "Package_TO_SOT_SMD:SOT-23" (id 2) (at 121.92 74.295 0)
       (effects (font (size 1.27 1.27) italic) (justify left) hide)
     )
