File: Kicad/maquina_compostaje/Opto_MB.kicad_sch (KiCad schematic)
At the start: 17 parts, among them Q5 BC328, Q6 BC328, Q7 BC328, Q8 BC328, U3 TLP281-4GB(F)

Commit message: inicio del ruteo
Parts:
- Q5, Q6, Q7, Q8: footprint Package_TO_SOT_THT:TO-92_Inline -> Package_TO_SOT_SMD:SOT-23
- U3: footprint (none) -> Package_SO:SO-16_5.3x10.2mm_P1.27mm
Connections:
- net GND: no longer Q5.1 (C), Q6.1 (C), Q7.1 (C), R22.2, R24.2, R26.2
- new net B2: Q7.1 (C), R26.2
- new net B3: Q6.1 (C), R24.2
- new net B4: Q5.1 (C), R22.2
Changed lines of the file:
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@@
   (junction (at 184.15 85.09) (diameter 0) (color 0 0 0 0)
   )
-  (junction (at 203.2 105.41) (diameter 0) (color 0 0 0 0)
-  )
-  (junction (at 203.2 85.09) (diameter 0) (color 0 0 0 0)
-  )
-  (junction (at 184.15 95.25) (diameter 0) (color 0 0 0 0)
-  )
   (junction (at 99.06 118.11) (diameter 0) (color 0 0 0 0)
   )
@@
   (junction (at 137.16 110.49) (diameter 0) (color 0 0 0 0)
   )
-  (junction (at 203.2 95.25) (diameter 0) (color 0 0 0 0)
-  )
-  (junction (at 165.1 105.41) (diameter 0) (color 0 0 0 0)
-  )
   (junction (at 165.1 118.11) (diameter 0) (color 0 0 0 0)
   )
@@
     (stroke (width 0) (type default) (color 0 0 0 0))
   )
-  (wire (pts (xy 203.2 85.09) (xy 203.2 95.25))
-    (stroke (width 0) (type default) (color 0 0 0 0))
-  )
-  (wire (pts (xy 203.2 57.15) (xy 228.6 57.15))
-    (stroke (width 0) (type default) (color 0 0 0 0))
-  )
-  (wire (pts (xy 146.05 105.41) (xy 146.05 106.68))
-    (stroke (width 0) (type default) (color 0 0 0 0))
-  )
   (wire (pts (xy 175.26 90.17) (xy 127 90.17))
     (stroke (width 0) (type default) (color 0 0 0 0))
@@
     (stroke (width 0) (type default) (color 0 0 0 0))
   )
-  (wire (pts (xy 146.05 105.41) (xy 165.1 105.41))
+  (wire (pts (xy 146.05 105.41) (xy 228.6 105.41))
     (stroke (width 0) (type default) (color 0 0 0 0))
   )
@@
     (stroke (width 0) (type default) (color 0 0 0 0))
   )
-  (wire (pts (xy 165.1 95.25) (xy 184.15 95.25))
+  (wire (pts (xy 165.1 95.25) (xy 228.6 95.25))
     (stroke (width 0) (type default) (color 0 0 0 0))
   )
@@
     (stroke (width 0) (type default) (color 0 0 0 0))
   )
-  (wire (pts (xy 228.6 105.41) (xy 203.2 105.41))
-    (stroke (width 0) (type default) (color 0 0 0 0))
-  )
   (wire (pts (xy 194.31 80.01) (xy 195.58 80.01))
     (stroke (width 0) (type default) (color 0 0 0 0))
@@
     (stroke (width 0) (type default) (color 0 0 0 0))
   )
-  (wire (pts (xy 228.6 95.25) (xy 203.2 95.25))
-    (stroke (width 0) (type default) (color 0 0 0 0))
-  )
   (wire (pts (xy 146.05 118.11) (xy 129.54 118.11))
     (stroke (width 0) (type default) (color 0 0 0 0))
@@
     (stroke (width 0) (type default) (color 0 0 0 0))
   )
-  (wire (pts (xy 184.15 95.25) (xy 203.2 95.25))
-    (stroke (width 0) (type default) (color 0 0 0 0))
-  )
   (wire (pts (xy 99.06 124.46) (xy 99.06 118.11))
     (stroke (width 0) (type default) (color 0 0 0 0))
   )
-  (wire (pts (xy 165.1 105.41) (xy 203.2 105.41))
-    (stroke (width 0) (type default) (color 0 0 0 0))
-  )
   (wire (pts (xy 129.54 97.79) (xy 129.54 107.95))
     (stroke (width 0) (type default) (color 0 0 0 0))
@@
     (stroke (width 0) (type default) (color 0 0 0 0))
   )
-  (wire (pts (xy 184.15 85.09) (xy 203.2 85.09))
-    (stroke (width 0) (type default) (color 0 0 0 0))
-  )
-  (wire (pts (xy 203.2 85.09) (xy 228.6 85.09))
+  (wire (pts (xy 184.15 85.09) (xy 228.6 85.09))
     (stroke (width 0) (type default) (color 0 0 0 0))
   )
@@
     (stroke (width 0) (type default) (color 0 0 0 0))
   )
-  (wire (pts (xy 203.2 105.41) (xy 203.2 118.11))
-    (stroke (width 0) (type default) (color 0 0 0 0))
-  )
-  (wire (pts (xy 203.2 95.25) (xy 203.2 105.41))
+  (wire (pts (xy 203.2 85.09) (xy 203.2 118.11))
     (stroke (width 0) (type default) (color 0 0 0 0))
   )
@@
   (hierarchical_label "M_B2" (shape input) (at 76.2 90.17 180)
     (effects (font (size 1.27 1.27)) (justify right))
-  )
-  (hierarchical_label "Vo_12V" (shape output) (at 228.6 57.15 0)
-    (effects (font (size 1.27 1.27)) (justify left))
   )
   (hierarchical_label "M_B3" (shape input) (at 76.2 100.33 180)
@@
     (property "Reference" "U3" (id 0) (at 115.57 73.2282 0))
     (property "Value" "TLP281-4GB(F)" (id 1) (at 115.57 75.5396 0))
-    (property "Footprint" "" (id 2) (at 114.3 97.79 0)
+    (property "Footprint" "Package_SO:SO-16_5.3x10.2mm_P1.27mm" (id 2) (at 114.3 97.79 0)
       (effects (font (size 1.27 1.27)) (justify left bottom) hide)
     )
@@
       (effects (font (size 1.27 1.27)) (justify left))
     )
-    (property "Footprint" "Package_TO_SOT_THT:TO-92_Inline" (id 2) (at 148.59 112.395 0)
+    (property "Footprint" "Package_TO_SOT_SMD:SOT-23" (id 2) (at 148.59 112.395 0)
       (effects (font (size 1.27 1.27) italic) (justify left) hide)
     )
@@
       (effects (font (size 1.27 1.27)) (justify left))
     )
-    (property "Footprint" "Package_TO_SOT_THT:TO-92_Inline" (id 2) (at 186.69 92.075 0)
+    (property "Footprint" "Package_TO_SOT_SMD:SOT-23" (id 2) (at 186.69 92.075 0)
       (effects (font (size 1.27 1.27) italic) (justify left) hide)
     )
@@
       (effects (font (size 1.27 1.27)) (justify left))
     )
-    (property "Footprint" "Package_TO_SOT_THT:TO-92_Inline" (id 2) (at 167.64 102.235 0)
+    (property "Footprint" "Package_TO_SOT_SMD:SOT-23" (id 2) (at 167.64 102.235 0)
       (effects (font (size 1.27 1.27) italic) (justify left) hide)
     )
@@
       (effects (font (size 1.27 1.27)) (justify left))
     )
-    (property "Footprint" "Package_TO_SOT_THT:TO-92_Inline" (id 2) (at 205.74 81.915 0)
+    (property "Footprint" "Package_TO_SOT_SMD:SOT-23" (id 2) (at 205.74 81.915 0)
       (effects (font (size 1.27 1.27) italic) (justify left) hide)
     )
