File: Kicad/maquina_compostaje/powersupply.kicad_sch (KiCad schematic)
At the start: 16 parts, among them J6 Barrel_Jack_MountingPin, U6 AMS1117-5.0, U7 AMS1117-3.3

Commit message: inicio del ruteo
Parts:
- D17: footprint Diode_THT:D_DO-41_SOD81_P10.16mm_Horizontal -> Diode_SMD:D_SOD-128
- U6: footprint AMS1117-5:SOT229P700X180-4N -> Package_TO_SOT_SMD:SOT-223
- U7: footprint AMS1117-3:SOT229P700X180-4N -> Package_TO_SOT_SMD:SOT-223
Connections:
- net GND: now also C12.2
Changed lines of the file:
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@@
     (stroke (width 0) (type default) (color 0 0 0 0))
   )
-  (wire (pts (xy 214.63 57.15) (xy 214.63 69.85))
+  (wire (pts (xy 214.63 57.15) (xy 214.63 72.39))
     (stroke (width 0) (type default) (color 0 0 0 0))
   )
@@
   (hierarchical_label "3.3V" (shape input) (at 243.84 40.64 90)
     (effects (font (size 1.27 1.27)) (justify left))
+  )
+  (symbol (lib_id "power:GND") (at 214.63 72.39 0) (unit 1)
+    (in_bom yes) (on_board yes) (fields_autoplaced)
+    (property "Reference" "#PWR01" (id 0) (at 214.63 78.74 0)
+      (effects (font (size 1.27 1.27)) hide)
+    )
+    (property "Value" "GND" (id 1) (at 214.63 77.47 0))
+    (property "Footprint" "" (id 2) (at 214.63 72.39 0)
+      (effects (font (size 1.27 1.27)) hide)
+    )
+    (property "Datasheet" "" (id 3) (at 214.63 72.39 0)
+      (effects (font (size 1.27 1.27)) hide)
+    )
+    (pin "1")
   )
   (symbol (lib_id "Device:C") (at 248.92 50.8 0) (unit 1)
@@
     (property "Reference" "D17" (id 0) (at 59.69 36.83 0))
     (property "Value" "1N4002" (id 1) (at 59.69 39.37 0))
-    (property "Footprint" "Diode_THT:D_DO-41_SOD81_P10.16mm_Horizontal" (id 2) (at 59.69 38.735 0)
+    (property "Footprint" "Diode_SMD:D_SOD-128" (id 2) (at 59.69 38.735 0)
       (effects (font (size 1.27 1.27)) hide)
     )
@@
     (property "Reference" "U6" (id 0) (at 110.49 35.56 0))
     (property "Value" "AMS1117-5.0" (id 1) (at 110.49 38.1 0))
-    (property "Footprint" "AMS1117-5:SOT229P700X180-4N" (id 2) (at 110.49 45.72 0)
+    (property "Footprint" "Package_TO_SOT_SMD:SOT-223" (id 2) (at 110.49 45.72 0)
       (effects (font (size 1.27 1.27)) (justify left bottom) hide)
     )
@@
     (property "Reference" "U7" (id 0) (at 193.04 35.56 0))
     (property "Value" "AMS1117-3.3" (id 1) (at 193.04 38.1 0))
-    (property "Footprint" "AMS1117-3:SOT229P700X180-4N" (id 2) (at 193.04 45.72 0)
-      (effects (font (size 1.27 1.27)) (justify left bottom) hide)
-    )
+    (property "Footprint" "Package_TO_SOT_SMD:SOT-223" (id 2) (at 193.04 45.72 0)
+      (effects (font (size 1.27 1.27)) (justify left bottom) hide)
+    )
