File: Kicad/maquina_compostaje/Serial_USB.kicad_sch (KiCad schematic)
At the start: 1 part, among them J7 Conn_01x06

Commit message: se agregaron componentes en la parte inferior de la placa
Parts:
- J7: value Conn_01x06 -> SERIAL_USB
Changed lines of the file:
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@@
       (effects (font (size 1.27 1.27)) (justify left))
     )
-    (property "Value" "Conn_01x06" (id 1) (at 41.91 29.2099 0)
+    (property "Value" "SERIAL_USB" (id 1) (at 41.91 29.2099 0)
       (effects (font (size 1.27 1.27)) (justify left))
     )
